File: hardware/esp8266_temp_monitor.sch (EAGLE design)
At the start: 27 parts, among them CN1 Power, IC1 REG1117, SW1 Reset, SW2 Config, U1 ESP-12

Commit message: Fixed minor circuit diagram error
Modified LED description
Parts:
- LED2: value Prog (AMBER) -> Run (GREEN)
- LED3: value Run (GREEN) -> Prog (AMBER)
Connections:
- removed net LED_RUN: LED3.A, R7.2
- new net LED_OPERATE: LED2.A, R6.2
- net LED_PROG: now also LED3.A, R7.2; no longer LED2.A, R6.2
Changed lines of the file:
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@@
 <part name="R7" library="resistor" deviceset="R-EU_" device="M0805" value="470"/>
 <part name="LED1" library="led" deviceset="LED" device="5MM" value="Fault (RED)"/>
-<part name="LED2" library="led" deviceset="LED" device="5MM" value="Prog (AMBER)"/>
-<part name="LED3" library="led" deviceset="LED" device="5MM" value="Run (GREEN)"/>
+<part name="LED2" library="led" deviceset="LED" device="5MM" value="Run (GREEN)"/>
+<part name="LED3" library="led" deviceset="LED" device="5MM" value="Prog (AMBER)"/>
 <part name="R8" library="resistor" deviceset="R-EU_" device="M0805" value="5.1K 1%"/>
 <part name="R9" library="resistor" deviceset="R-EU_" device="M0805" value="1K 1%"/>
@@
 </segment>
 </net>
-<net name="LED_PROG" class="0">
+<net name="LED_OPERATE" class="0">
 <segment>
 <pinref part="R6" gate="G$1" pin="2"/>
@@
 </segment>
 </net>
-<net name="LED_RUN" class="0">
+<net name="LED_PROG" class="0">
 <segment>
 <pinref part="R7" gate="G$1" pin="2"/>
